File: momo.kicad_pcb (KiCad board)
At the start: 2 copper layers, 228.1 x 85.4 mm, 221 parts, among them J1 USB C, Q1 2N7002, Q2 2N7002, Q3 2N7002, SW1 MX_SW_HS, SW10 MX_SW_HS, SW11 MX_SW_HS, SW12 MX_SW_HS, SW13 MX_SW_HS, SW14 MX_SW_HS, SW15 MX_SW_HS, SW16 MX_SW_HS, SW17 MX_SW_HS, SW18 MX_SW_HS, SW19 MX_SW_HS, SW2 MX_SW_HS, SW20 MX_SW_HS, SW21 MX_SW_HS, SW22 MX_SW_HS, SW23 MX_SW_HS, SW24 MX_SW_HS, SW25 MX_SW_HS, SW26 MX_SW_HS, SW27 MX_SW_HS, SW28 MX_SW_HS, SW29 MX_SW_HS, SW3 MX_SW_HS, SW30 MX_SW_HS, SW31 MX_SW_HS, SW32 MX_SW_HS, SW33 MX_SW_HS, SW34 MX_SW_HS, SW35 MX_SW_HS, SW36 MX_SW_HS, SW37 MX_SW_HS, SW38 MX_SW_HS, SW39 MX_SW_HS, SW4 MX_SW_HS, SW40 MX_SW_HS, SW41 MX_SW_HS, SW42 MX_SW_HS, SW43 MX_SW_HS, SW44 MX_SW_HS, SW45 MX_SW_HS, SW46 MX_SW_HS, SW47 MX_SW_HS, SW48 MX_SW_HS, SW5 MX_SW_HS, SW6 MX_SW_HS, SW7 MX_SW_HS, SW8 MX_SW_HS, SW9 MX_SW_HS, U1 WeAct-RP2040-Pico

Commit message: Added i2c pins
Parts:
- added J2: Rows, Connector_PinHeader_2.54mm:PinHeader_1x04_P2.54mm_Vertical, F.Cu at (60.5, 102.9)
- added J3: I2C, Connector_PinHeader_2.54mm:PinHeader_1x04_P2.54mm_Vertical, F.Cu at (251.2, 102.6)
- added J4: Columns, Connector_PinHeader_2.54mm:PinHeader_1x12_P2.54mm_Vertical, F.Cu at (97.3, 102.4)
- C1, C2, C3, C4, C5, C6, C7, C8, C9: footprint keyboard_parts:C_1608 -> Capacitor_SMD:C_1206_3216Metric_Pad1.33x1.80mm_HandSolder
- moved Q1 113.8 mm to (155.0, 122.2)
- moved R52 113.8 mm to (166.7, 123.5)
- moved R49 113.8 mm to (166.7, 121.0)
- moved R30 18.4 mm to (145.9, 122.2), turned to 180 degrees
- moved C9 0.35 mm to (70.1, 122.4), turned to -90 degrees
- moved C8 0.32 mm to (127.3, 122.4), turned to -90 degrees
- moved C4 0.32 mm to (222.5, 103.4), turned to -90 degrees
- moved C1 0.30 mm to (241.6, 84.3), turned to -90 degrees
- moved C6 0.30 mm to (241.6, 122.4), turned to -90 degrees
- moved C7 0.30 mm to (184.4, 122.4), turned to -90 degrees
- moved C2 0.25 mm to (127.3, 84.3), turned to -90 degrees
- moved C5 0.06 mm to (88.9, 103.2), turned to -90 degrees
- moved C3 0.06 mm to (69.8, 84.1), turned to -90 degrees
Other:
- outline, holes or cut-outs redrawn
- board text added: "1"
- board text added: "10"
- board text added: "11"
- board text added: "2"
- board text added: "3"
- board text added: "4"
- board text added: "5"
- board text added: "6"
- board text added: "7"
- board text added: "8"
- board text added: "9"
- board text added: "COL"
- board text added: "Calebe94"
- board text added: "GND"
- board text added: "MOMO Keyboard v1"
- board text added: "O"
- board text added: "ROW"
- board text added: "SCL"
- board text added: "SDA"
- board text added: "SW1"
- board text added: "SW10"
- board text added: "SW11"
- board text added: "SW12"
- board text added: "SW13"
- board text added: "SW14"
- board text added: "SW15"
- board text added: "SW16"
- board text added: "SW17"
- board text added: "SW18"
- board text added: "SW19"
- board text added: "SW2"
- board text added: "SW20"
- board text added: "SW21"
- board text added: "SW22"
- board text added: "SW23"
- board text added: "SW24"
- board text added: "SW25"
- board text added: "SW26"
- board text added: "SW27"
- board text added: "SW28"
- board text added: "SW29"
- board text added: "SW3"
- board text added: "SW30"
- board text added: "SW31"
- board text added: "SW32"
- board text added: "SW33"
- board text added: "SW34"
- board text added: "SW35"
- board text added: "SW36"
- board text added: "SW37"
- board text added: "SW38"
- board text added: "SW39"
- board text added: "SW4"
- board text added: "SW40"
- board text added: "SW41"
- board text added: "SW42"
- board text added: "SW43"
- board text added: "SW44"
- board text added: "SW45"
- board text added: "SW46"
- board text added: "SW47"
- board text added: "SW48"
- board text added: "SW5"
- board text added: "SW6"
- board text added: "SW7"
- board text added: "SW8"
- board text added: "SW9"
- board text added: "VCC"
- board text added: "calebe.dev.br"
