File: underglow.kicad_sch (KiCad schematic)
At the start: 18 parts

Commit message: Pin wiring
Parts:
- C1, C2, C3, C4, C5, C6, C7, C8, C9: renamed from C?; footprint (none) -> keyboard_parts:C_1608
- gave numbers to parts that had none: 9

Commit message: Added i2c pins
Parts:
- C1, C2, C3, C4, C5, C6, C7, C8, C9: footprint keyboard_parts:C_1608 -> Capacitor_SMD:C_1206_3216Metric_Pad1.33x1.80mm_HandSolder
Changed lines of the file:
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@@
       (effects (font (size 1.27 1.27)) (justify left))
     )
-    (property "Footprint" "keyboard_parts:C_1608" (id 2) (at 173.9392 91.44 0)
+    (property "Footprint" "Capacitor_SMD:C_1206_3216Metric_Pad1.33x1.80mm_HandSolder" (id 2) (at 173.9392 91.44 0)
       (effects (font (size 1.27 1.27)) hide)
     )
@@
       (effects (font (size 1.27 1.27)) (justify left))
     )
-    (property "Footprint" "keyboard_parts:C_1608" (id 2) (at 49.7332 39.878 0)
+    (property "Footprint" "Capacitor_SMD:C_1206_3216Metric_Pad1.33x1.80mm_HandSolder" (id 2) (at 49.7332 39.878 0)
       (effects (font (size 1.27 1.27)) hide)
     )
@@
       (effects (font (size 1.27 1.27)) (justify left))
     )
-    (property "Footprint" "keyboard_parts:C_1608" (id 2) (at 80.9752 91.44 0)
+    (property "Footprint" "Capacitor_SMD:C_1206_3216Metric_Pad1.33x1.80mm_HandSolder" (id 2) (at 80.9752 91.44 0)
       (effects (font (size 1.27 1.27)) hide)
     )
@@
       (effects (font (size 1.27 1.27)) (justify left))
     )
-    (property "Footprint" "keyboard_parts:C_1608" (id 2) (at 111.7092 39.878 0)
+    (property "Footprint" "Capacitor_SMD:C_1206_3216Metric_Pad1.33x1.80mm_HandSolder" (id 2) (at 111.7092 39.878 0)
       (effects (font (size 1.27 1.27)) hide)
     )
@@
       (effects (font (size 1.27 1.27)) (justify left))
     )
-    (property "Footprint" "keyboard_parts:C_1608" (id 2) (at 80.7212 39.878 0)
+    (property "Footprint" "Capacitor_SMD:C_1206_3216Metric_Pad1.33x1.80mm_HandSolder" (id 2) (at 80.7212 39.878 0)
       (effects (font (size 1.27 1.27)) hide)
     )
@@
       (effects (font (size 1.27 1.27)) (justify left))
     )
-    (property "Footprint" "keyboard_parts:C_1608" (id 2) (at 111.9632 91.44 0)
+    (property "Footprint" "Capacitor_SMD:C_1206_3216Metric_Pad1.33x1.80mm_HandSolder" (id 2) (at 111.9632 91.44 0)
       (effects (font (size 1.27 1.27)) hide)
     )
@@
       (effects (font (size 1.27 1.27)) (justify left))
     )
-    (property "Footprint" "keyboard_parts:C_1608" (id 2) (at 142.9512 91.44 0)
+    (property "Footprint" "Capacitor_SMD:C_1206_3216Metric_Pad1.33x1.80mm_HandSolder" (id 2) (at 142.9512 91.44 0)
       (effects (font (size 1.27 1.27)) hide)
     )
@@
       (effects (font (size 1.27 1.27)) (justify left))
     )
-    (property "Footprint" "keyboard_parts:C_1608" (id 2) (at 49.9872 91.44 0)
+    (property "Footprint" "Capacitor_SMD:C_1206_3216Metric_Pad1.33x1.80mm_HandSolder" (id 2) (at 49.9872 91.44 0)
       (effects (font (size 1.27 1.27)) hide)
     )
@@
       (effects (font (size 1.27 1.27)) (justify left))
     )
-    (property "Footprint" "keyboard_parts:C_1608" (id 2) (at 142.6972 39.878 0)
-      (effects (font (size 1.27 1.27)) hide)
-    )
+    (property "Footprint" "Capacitor_SMD:C_1206_3216Metric_Pad1.33x1.80mm_HandSolder" (id 2) (at 142.6972 39.878 0)
+      (effects (font (size 1.27 1.27)) hide)
+    )

Commit message: Routed components
Connections:
- net UNDERGLOW_TO_BACKLIGHT: now reaches D57.2 (DOUT)
Changed lines of the file:
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@@
+    (stroke (width 0) (type default) (color 0 0 0 0))
+  )
+  (wire (pts (xy 191.516 102.108) (xy 193.294 102.108))
     (stroke (width 0) (type default) (color 0 0 0 0))
   )
@@
     )
   )
+  (global_label "UNDERGLOW_TO_BACKLIGHT" (shape input) (at 193.294 102.108 0) (fields_autoplaced)
+    (effects (font (size 1.27 1.27)) (justify left))
+    (property "Referências entre as folhas" "${INTERSHEET_REFS}" (id 0) (at 221.47 102.0286 0)
+      (effects (font (size 1.27 1.27)) (justify left) hide)
+    )
+  )
